Commit message: Updated DG-5F right URDF to simplify collision mesh. Added configuration for GeoRT training

File: assets/dg5f_right/dg5f_right.urdf (robot description, URDF)
Before this commit: robot dg5f_right, 28 links, 27 joints
Links:
- link rl_dg_1_1: geometry collision box size=0.0626 0.0190 0.0287; visual mesh filename=meshes/visual/rl_dg_1_1.dae
- link rl_dg_1_2: geometry collision box size=0.0224 0.044 0.0224; visual mesh filename=meshes/visual/rl_dg_1_2.dae
- link rl_dg_1_3: geometry collision box size=0.0224 0.0547639 0.0190; visual mesh filename=meshes/visual/rl_dg_1_3.dae
- link rl_dg_1_4: geometry collision mesh filename=meshes/collision/rl_dg_1_4_c.obj; visual mesh filename=meshes/visual/rl_dg_1_4.dae
- link rl_dg_1_tip: geometry collision mesh filename=meshes/collision/rl_dg_1_tip_c.obj; visual mesh filename=meshes/visual/rl_dg_1_tip.dae
- link rl_dg_2_1: geometry collision box size=0.042749165557324886 0.0239 0.046708067413419485; visual mesh filename=meshes/visual/rl_dg_2_1.dae
- link rl_dg_2_2: geometry collision box size=0.0190 0.0224 0.0547639; visual mesh filename=meshes/visual/rl_dg_2_2.dae
- link rl_dg_2_3: geometry collision box size=0.0190 0.0224 0.0547639; visual mesh filename=meshes/visual/rl_dg_2_3.dae
- link rl_dg_2_4: geometry collision mesh filename=meshes/collision/rl_dg_2_4_c.obj; visual mesh filename=meshes/visual/rl_dg_2_4.dae
- link rl_dg_2_tip: geometry collision mesh filename=meshes/collision/rl_dg_2_tip_c.obj; visual mesh filename=meshes/visual/rl_dg_2_tip.dae
- link rl_dg_3_1: geometry collision box size=0.04273 0.0224 0.0466; visual mesh filename=meshes/visual/rl_dg_3_1.dae
- link rl_dg_3_2: geometry collision box size=0.0190 0.0224 0.0547639; visual mesh filename=meshes/visual/rl_dg_3_2.dae
- link rl_dg_3_3: geometry collision box size=0.0190 0.0224 0.0547639; visual mesh filename=meshes/visual/rl_dg_3_3.dae
- link rl_dg_3_4: geometry collision mesh filename=meshes/collision/rl_dg_3_4_c.obj; visual mesh filename=meshes/visual/rl_dg_3_4.dae
- link rl_dg_3_tip: geometry collision mesh filename=meshes/collision/rl_dg_3_tip_c.obj; visual mesh filename=meshes/visual/rl_dg_3_tip.dae
- link rl_dg_4_1: geometry collision box size=0.04275 0.0239 0.0467; visual mesh filename=meshes/visual/rl_dg_4_1.dae
- link rl_dg_4_2: geometry collision box size=0.0190 0.0224 0.0547639; visual mesh filename=meshes/visual/rl_dg_4_2.dae
- link rl_dg_4_3: geometry collision box size=0.0190 0.0224 0.0547639; visual mesh filename=meshes/visual/rl_dg_4_3.dae
- link rl_dg_4_4: geometry collision mesh filename=meshes/collision/rl_dg_4_4_c.obj; visual mesh filename=meshes/visual/rl_dg_4_4.dae
- link rl_dg_4_tip: geometry collision mesh filename=meshes/collision/rl_dg_4_tip_c.obj; visual mesh filename=meshes/visual/rl_dg_4_tip.dae
- link rl_dg_5_1: geometry collision box size=0.03444028086960316 0.04645590577274561 0.060140796937048435; visual mesh filename=meshes/visual/rl_dg_5_1.dae
- link rl_dg_5_2: geometry collision box size=0.0224 0.0224 0.0440; visual mesh filename=meshes/visual/rl_dg_5_2.dae
- link rl_dg_5_3: geometry collision box size=0.0190 0.0224 0.0547639; visual mesh filename=meshes/visual/rl_dg_5_3.dae
- link rl_dg_5_4: geometry collision mesh filename=meshes/collision/rl_dg_5_4_c.obj; visual mesh filename=meshes/visual/rl_dg_5_4.dae
- link rl_dg_5_tip: geometry collision mesh filename=meshes/collision/rl_dg_5_tip_c.obj; visual mesh filename=meshes/visual/rl_dg_5_tip.dae
- link rl_dg_base: geometry collision box size=0.0700 0.0705 0.0920307; visual mesh filename=meshes/visual/rl_dg_base.dae
- link rl_dg_mount: geometry collision box size=0.062 0.06195 0.012; visual mesh filename=meshes/visual/rl_dg_mount.dae
- link rl_dg_palm: geometry collision box size=0.06403926014900208 0.08234254270792007 0.09909999370574955; visual mesh filename=meshes/visual/rl_dg_palm.dae
