Commit message: feat: Add dg4f/dg5f support and improve trainer
- Add collision meshes for dg5f_right fingers (4 & 5)
- Add dg4f_right configuration file
- Add FK model checkpoints for dg4f_right and dg5f_right
- Improve model architecture with additional hidden layers
- Add logging system to save CLI output to output.log in checkpoint folders
- Add configurable save_every parameter for checkpointing
- Add FK training epoch configuration
- Fix dataset import typo
- Add fingertip geometry analysis utilities for offset calibration

File: assets/dg5f_right/dg4f_right.urdf (robot description, URDF)
Before this commit: robot dg5f_right, 28 links, 27 joints
Joints:
- joint rj_dg_3_2: limit lower=0.0 upper=1.9547687622336491 effort=7.5 velocity=3.141592653589793 -> lower=-0.1 upper=1.9547687622336491 effort=7.5 velocity=3.141592653589793
- joint rj_dg_5_1: axis 0 0 1 -> (none); limit lower=-0.017453292519943295 upper=1.0471975511965976 effort=7.5 velocity=3.141592653589793 -> (none); type revolute -> fixed
- joint rj_dg_5_2: axis 1 0 0 -> (none); limit lower=-0.4188790204786391 upper=0.6108652381980153 effort=7.5 velocity=3.141592653589793 -> (none); type revolute -> fixed
- joint rj_dg_5_3: axis 0 1 0 -> (none); limit lower=-0.1 upper=1.5707963267948966 effort=7.5 velocity=3.141592653589793 -> (none); type revolute -> fixed
- joint rj_dg_5_4: axis 0 1 0 -> (none); limit lower=-0.1 upper=1.5707963267948966 effort=7.5 velocity=3.141592653589793 -> (none); type revolute -> fixed
